File: Electronics/Connectors.kicad_sch (KiCad schematic)
At the start: 60 parts, among them J501 Switches, J502 Motor Con, J503 Hall Sensor, Q501 BC817, U501 ‎ACHS-7124-000E‎, U502 LM393, U503 74AHC08, U504 MCP6001-OT

Commit message: Changed capacitor to multi footprint version. Added parallel diodes to MOSFET gate resistors to improve Turn-OFF time.
Changed lines of the file:
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@@
     )
     (property "Value" "Current Out" (id 1) (at 142.113 95.2116 0)
-      (effects (font (size 1.27 1.27)) (justify left) hide)
+      (effects (font (size 1.27 1.27)) (justify left))
     )
     (property "Footprint" "TestPoint:TestPoint_Pad_D1.0mm" (id 2) (at 146.05 93.345 0)
@@
     (property "Reference" "TP502" (id 0) (at 134.62 112.7275 90))
     (property "Value" "Current Out Att" (id 1) (at 136.4866 115.443 0)
-      (effects (font (size 1.27 1.27)) (justify left) hide)
+      (effects (font (size 1.27 1.27)) (justify left))
     )
     (property "Footprint" "TestPoint:TestPoint_Pad_D1.0mm" (id 2) (at 134.62 119.38 0)
@@
       (effects (font (size 1.27 1.27)) hide)
     )
-    (property "Value" "PWR_FLAG" (id 1) (at 185.42 19.2555 0)
-      (effects (font (size 1.27 1.27)) hide)
-    )
+    (property "Value" "PWR_FLAG" (id 1) (at 185.42 19.2555 0))
     (property "Footprint" "" (id 2) (at 185.42 22.86 0)
       (effects (font (size 1.27 1.27)) hide)
@@
       (effects (font (size 1.27 1.27)) hide)
     )
-    (property "Value" "PWR_FLAG" (id 1) (at 217.805 23.7005 0)
-      (effects (font (size 1.27 1.27)) hide)
-    )
+    (property "Value" "PWR_FLAG" (id 1) (at 217.805 23.7005 0))
     (property "Footprint" "" (id 2) (at 217.805 27.305 0)
       (effects (font (size 1.27 1.27)) hide)
@@
     )
     (property "Value" "GND" (id 1) (at 220.853 92.0366 0)
-      (effects (font (size 1.27 1.27)) (justify left) hide)
+      (effects (font (size 1.27 1.27)) (justify left))
     )
     (property "Footprint" "TestPoint:TestPoint_Pad_1.5x1.5mm" (id 2) (at 224.79 90.17 0)
@@
     )
     (property "Value" "Current Out AMP" (id 1) (at 171.577 116.0396 0)
-      (effects (font (size 1.27 1.27)) (justify left) hide)
+      (effects (font (size 1.27 1.27)) (justify left))
     )
     (property "Footprint" "TestPoint:TestPoint_Pad_D1.0mm" (id 2) (at 175.26 117.475 0)
@@
     )
     (property "Value" "GND" (id 1) (at 171.958 106.6416 0)
-      (effects (font (size 1.27 1.27)) (justify left) hide)
+      (effects (font (size 1.27 1.27)) (justify left))
     )
     (property "Footprint" "TestPoint:TestPoint_Pad_1.5x1.5mm" (id 2) (at 175.895 104.775 0)
@@
     )
     (property "Value" "GND" (id 1) (at 131.953 102.8316 0)
-      (effects (font (size 1.27 1.27)) (justify left) hide)
+      (effects (font (size 1.27 1.27)) (justify left))
     )
     (property "Footprint" "TestPoint:TestPoint_Pad_1.5x1.5mm" (id 2) (at 135.89 100.965 0)

Commit message: Manufacturing commit of PCB
Connections:
- net Limit_1: no longer D503.1 (K)
- net Limit_2: no longer D504.1 (K)
- net at C501.1, J501.1 (Pin_1), R501.1: now also D503.1 (K)
- net at C502.1, J501.3 (Pin_3), R502.1: now also D504.1 (K)
Other:
- moved on the sheet: D503, D504, R521, R522
