File: Electronics/hbridge.kicad_sch (KiCad schematic)
At the start: 37 parts, among them Q201 IRLZ44N, Q202 IRLIZ44N, Q203 IRLZ44N, Q204 IRLIZ44N, Q205 IRLZ44N, Q206 IRLIZ44N, U201 74AHC08, U202 IR2101, U203 IR2101, U204 IR2101

Commit message: Layout improvements
Signed-off-by: Aki Kuusela <git@findersee.fi>
Parts:
- U201: value 74AHC08 -> 74LS08; footprint Package_SO:SSOP-14_5.3x6.2mm_P0.65mm -> Package_SO:SO-14_3.9x8.65mm_P1.27mm
Other:
- company: (none) -> findersee.fi
- title: (none) -> Motor Controller
- moved on the sheet: R213, U201A
Changed lines of the file:
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@@
 (kicad_sch (version 20211123) (generator eeschema)
   (paper "A4")
+  (title_block
+    (title "Motor Controller")
+    (date "2022-02-18")
+    (rev "1.0")
+    (company "findersee.fi")
+  )
   (junction (at 152.4 113.03) (diameter 0) (color 0 0 0 0)
   )
@@
   (junction (at 116.84 129.54) (diameter 0) (color 0 0 0 0)
   )
-  (junction (at 27.94 43.18) (diameter 0) (color 0 0 0 0)
+  (junction (at 34.29 43.18) (diameter 0) (color 0 0 0 0)
   )
   (junction (at 116.84 135.89) (diameter 0) (color 0 0 0 0)
@@
   (junction (at 116.84 44.45) (diameter 0) (color 0 0 0 0)
   )
-  (junction (at 27.94 88.9) (diameter 0) (color 0 0 0 0)
+  (junction (at 34.29 88.9) (diameter 0) (color 0 0 0 0)
   )
   (junction (at 194.31 97.79) (diameter 0) (color 0 0 0 0)
@@
   (junction (at 116.84 67.31) (diameter 0) (color 0 0 0 0)
   )
-  (junction (at 27.94 128.27) (diameter 0) (color 0 0 0 0)
+  (junction (at 34.29 128.27) (diameter 0) (color 0 0 0 0)
   )
   (junction (at 222.25 96.52) (diameter 0) (color 0 0 0 0)
@@
     (stroke (width 0) (type default) (color 0 0 0 0))
   )
-  (wire (pts (xy 27.94 88.9) (xy 27.94 107.95))
+  (wire (pts (xy 34.29 88.9) (xy 34.29 107.95))
     (stroke (width 0) (type default) (color 0 0 0 0))
   )
@@
     (stroke (width 0) (type default) (color 0 0 0 0))
   )
-  (wire (pts (xy 25.4 48.26) (xy 31.75 48.26))
+  (wire (pts (xy 21.59 48.26) (xy 36.83 48.26))
     (stroke (width 0) (type default) (color 0 0 0 0))
   )
@@
     (stroke (width 0) (type default) (color 0 0 0 0))
   )
-  (wire (pts (xy 27.94 43.18) (xy 27.94 88.9))
+  (wire (pts (xy 34.29 43.18) (xy 34.29 88.9))
     (stroke (width 0) (type default) (color 0 0 0 0))
   )
@@
     (stroke (width 0) (type default) (color 0 0 0 0))
   )
-  (wire (pts (xy 25.4 43.18) (xy 27.94 43.18))
+  (wire (pts (xy 21.59 43.18) (xy 34.29 43.18))
     (stroke (width 0) (type default) (color 0 0 0 0))
   )
@@
     (stroke (width 0) (type default) (color 0 0 0 0))
   )
-  (wire (pts (xy 46.99 45.72) (xy 69.85 45.72))
+  (wire (pts (xy 52.07 45.72) (xy 69.85 45.72))
     (stroke (width 0) (type default) (color 0 0 0 0))
   )
@@
     (stroke (width 0) (type default) (color 0 0 0 0))
   )
-  (wire (pts (xy 27.94 113.03) (xy 27.94 128.27))
+  (wire (pts (xy 34.29 113.03) (xy 34.29 128.27))
     (stroke (width 0) (type default) (color 0 0 0 0))
   )
@@
     (stroke (width 0) (type default) (color 0 0 0 0))
   )
-  (wire (pts (xy 27.94 128.27) (xy 36.83 128.27))
+  (wire (pts (xy 34.29 128.27) (xy 36.83 128.27))
     (stroke (width 0) (type default) (color 0 0 0 0))
   )
@@
     (stroke (width 0) (type default) (color 0 0 0 0))
   )
-  (wire (pts (xy 27.94 43.18) (xy 31.75 43.18))
+  (wire (pts (xy 34.29 43.18) (xy 36.83 43.18))
     (stroke (width 0) (type default) (color 0 0 0 0))
   )
@@
     (stroke (width 0) (type default) (color 0 0 0 0))
   )
-  (wire (pts (xy 22.86 128.27) (xy 27.94 128.27))
+  (wire (pts (xy 22.86 128.27) (xy 34.29 128.27))
     (stroke (width 0) (type default) (color 0 0 0 0))
   )
@@
     (stroke (width 0) (type default) (color 0 0 0 0))
   )
-  (wire (pts (xy 27.94 88.9) (xy 152.4 88.9))
+  (wire (pts (xy 34.29 88.9) (xy 152.4 88.9))
     (stroke (width 0) (type default) (color 0 0 0 0))
   )
@@
     (effects (font (size 1.27 1.27)) (justify left))
   )
-  (hierarchical_label "A LIMIT" (shape input) (at 25.4 48.26 180)
+  (hierarchical_label "A LIMIT" (shape input) (at 21.59 48.26 180)
     (effects (font (size 1.27 1.27)) (justify right))
   )
@@
     (effects (font (size 1.27 1.27)) (justify left))
   )
-  (hierarchical_label "HIN A" (shape input) (at 25.4 43.18 180)
+  (hierarchical_label "HIN A" (shape input) (at 21.59 43.18 180)
     (effects (font (size 1.27 1.27)) (justify right))
   )
@@
     (pin "2")
   )
-  (symbol (lib_id "Device:R_Small") (at 27.94 110.49 0) (mirror x) (unit 1)
-    (in_bom yes) (on_board yes) (fields_autoplaced)
-    (property "Reference" "R213" (id 0) (at 26.4414 109.5815 0)
-      (effects (font (size 1.27 1.27)) (justify right))
-    )
-    (property "Value" "0" (id 1) (at 26.4414 112.3566 0)
-      (effects (font (size 1.27 1.27)) (justify right))
-    )
-    (property "Footprint" "Resistor_SMD:R_0603_1608Metric_Pad0.98x0.95mm_HandSolder" (id 2) (at 27.94 110.49 0)
-      (effects (font (size 1.27 1.27)) hide)
-    )
-    (property "Datasheet" "~" (id 3) (at 27.94 110.49 0)
+  (symbol (lib_id "Device:R_Small") (at 34.29 110.49 0) (mirror x) (unit 1)
+    (in_bom yes) (on_board yes) (fields_autoplaced)
+    (property "Reference" "R213" (id 0) (at 32.7914 109.5815 0)
+      (effects (font (size 1.27 1.27)) (justify right))
+    )
+    (property "Value" "0" (id 1) (at 32.7914 112.3566 0)
+      (effects (font (size 1.27 1.27)) (justify right))
+    )
+    (property "Footprint" "Resistor_SMD:R_0603_1608Metric_Pad0.98x0.95mm_HandSolder" (id 2) (at 34.29 110.49 0)
+      (effects (font (size 1.27 1.27)) hide)
+    )
+    (property "Datasheet" "~" (id 3) (at 34.29 110.49 0)
       (effects (font (size 1.27 1.27)) hide)
     )
@@
   (symbol (lib_id "74xx:74LS08") (at 161.29 115.57 0) (unit 2)
     (in_bom yes) (on_board yes) (fields_autoplaced)
-    (property "Reference" "U201" (id 0) (at 161.29 107.7935 0))
-    (property "Value" "74AHC08" (id 1) (at 161.29 110.5686 0))
-    (property "Footprint" "Package_SO:SSOP-14_5.3x6.2mm_P0.65mm" (id 2) (at 161.29 115.57 0)
+    (property "Reference" "U201" (id 0) (at 161.29 106.68 0))
+    (property "Value" "74LS08" (id 1) (at 161.29 109.22 0))
+    (property "Footprint" "Package_SO:SO-14_3.9x8.65mm_P1.27mm" (id 2) (at 161.29 115.57 0)
       (effects (font (size 1.27 1.27)) hide)
     )
@@
     (in_bom yes) (on_board yes) (fields_autoplaced)
     (property "Reference" "U201" (id 0) (at 44.45 123.0335 0))
-    (property "Value" "74AHC08" (id 1) (at 44.45 125.8086 0))
-    (property "Footprint" "Package_SO:SSOP-14_5.3x6.2mm_P0.65mm" (id 2) (at 44.45 130.81 0)
+    (property "Value" "74LS08" (id 1) (at 44.45 125.8086 0))
+    (property "Footprint" "Package_SO:SO-14_3.9x8.65mm_P1.27mm" (id 2) (at 44.45 130.81 0)
       (effects (font (size 1.27 1.27)) hide)
     )
@@
       (effects (font (size 1.27 1.27)) (justify left))
     )
-    (property "Value" "74AHC08" (id 1) (at 272.542 41.2366 0)
-      (effects (font (size 1.27 1.27)) (justify left))
-    )
-    (property "Footprint" "Package_SO:SSOP-14_5.3x6.2mm_P0.65mm" (id 2) (at 266.7 39.37 0)
+    (property "Value" "74LS08" (id 1) (at 272.542 41.2366 0)
+      (effects (font (size 1.27 1.27)) (justify left))
+    )
+    (property "Footprint" "Package_SO:SO-14_3.9x8.65mm_P1.27mm" (id 2) (at 266.7 39.37 0)
       (effects (font (size 1.27 1.27)) hide)
     )
@@
     (in_bom yes) (on_board yes) (fields_autoplaced)
     (property "Reference" "U201" (id 0) (at 224.79 32.8635 0))
-    (property "Value" "74AHC08" (id 1) (at 224.79 35.6386 0))
-    (property "Footprint" "Package_SO:SSOP-14_5.3x6.2mm_P0.65mm" (id 2) (at 224.79 40.64 0)
+    (property "Value" "74LS08" (id 1) (at 224.79 35.6386 0))
+    (property "Footprint" "Package_SO:SO-14_3.9x8.65mm_P1.27mm" (id 2) (at 224.79 40.64 0)
       (effects (font (size 1.27 1.27)) hide)
     )
@@
     (pin "2")
   )
-  (symbol (lib_id "74xx:74LS08") (at 39.37 45.72 0) (unit 1)
-    (in_bom yes) (on_board yes) (fields_autoplaced)
-    (property "Reference" "U201" (id 0) (at 39.37 37.9435 0))
-    (property "Value" "74AHC08" (id 1) (at 39.37 40.7186 0))
-    (property "Footprint" "Package_SO:SSOP-14_5.3x6.2mm_P0.65mm" (id 2) (at 39.37 45.72 0)
-      (effects (font (size 1.27 1.27)) hide)
-    )
-    (property "Datasheet" "http://www.ti.com/lit/gpn/sn74LS08" (id 3) (at 39.37 45.72 0)
-      (effects (font (size 1.27 1.27)) hide)
-    )
+  (symbol (lib_id "74xx:74LS08") (at 44.45 45.72 0) (unit 1)
+    (in_bom yes) (on_board yes) (fields_autoplaced)
+    (property "Reference" "U201" (id 0) (at 44.45 37.9435 0))
+    (property "Value" "74LS08" (id 1) (at 44.45 40.7186 0))
+    (property "Footprint" "Package_SO:SO-14_3.9x8.65mm_P1.27mm" (id 2) (at 44.45 45.72 0)
+      (effects (font (size 1.27 1.27)) hide)
+    )
+    (property "Datasheet" "http://www.ti.com/lit/gpn/sn74LS08" (id 3) (at 44.45 45.72 0)
+      (effects (font (size 1.27 1.27)) hide)
+    )

Commit message: Changed capacitor to multi footprint version. Added parallel diodes to MOSFET gate resistors to improve Turn-OFF time.
Parts:
- added D204, D205, D206, D207, D208, D209: 1N5819, Diode_SMD:D_SOD-123, symbol Diode:1N5819
- C206, C207, C210: value C -> 100u; footprint Capacitor_THT:CP_Radial_D10.0mm_P5.00mm -> Findersee_parts:CP_Radial_D12.5mm_P3.5-5.0mm
Connections:
- net at Q201.1 (G), R203.2, R207.2: now also D206.2 (A)
- net at Q204.1 (G), R202.1, R206.2: now also D205.2 (A)
- net at Q205.1 (G), R210.2, R212.1: now also D209.2 (A)
- net at R210.1, U204.7 (HO): now also D209.1 (K)
- net at Q203.1 (G), R204.2, R208.1: now also D207.2 (A)
- net at Q202.1 (G), R201.1, R205.2: now also D204.2 (A)
- net at R201.2, U202.5 (LO): now also D204.1 (K)
- net at R202.2, U203.5 (LO): now also D205.1 (K)
- net at R204.1, U203.7 (HO): now also D207.1 (K)
- net at R209.2, U204.5 (LO): now also D208.1 (K)
- net at R203.1, U202.7 (HO): now also D206.1 (K)
- net at Q206.1 (G), R209.1, R211.2: now also D208.2 (A)
Other:
- moved on the sheet: C205, C207, C208, C209, C210, D203, Q205, Q206, R201, R202, R203, R204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

Commit message: Manufacturing commit of PCB
Parts:
- added C211: 100n, Capacitor_SMD:C_0603_1608Metric_Pad1.08x0.95mm_HandSolder, symbol Device:C
- added R215, R216, R217, R218: 0, Resistor_SMD:R_0603_1608Metric_Pad0.98x0.95mm_HandSolder, symbol Device:R_Small
- added U205: 74LS08, Package_SO:SO-14_3.9x8.65mm_P1.27mm, symbol 74xx:74LS08
- C201: value C -> 100n
Connections:
- net +3V3: now also C211.1, U205.14 (VCC); no longer U201.12, U201.13
- net GND: now also U201.12, U201.13, C211.2, U205.10, U205.7 (GND), U205.9
- net HIN A: now also R218.2
- net LIN A: now also R217.2, R218.1, U205.1, U205.13, U205.4; no longer U202.3 (LIN)
- net LIN B: now also R215.2, U205.5; no longer U203.3 (LIN)
- net LIN C: now also R216.2, U205.12; no longer U204.3 (LIN)
- net C LIMIT renamed C CTRL
- new net: R215.1, U203.3 (LIN), U205.6
- new net: R217.1, U202.3 (LIN), U205.3
- new net: R216.1, U204.3 (LIN), U205.11
- new net A CTRL: U205.2
- no-connect marks 1 -> 2
Other:
- moved on the sheet: C201, R213, U201D
