File: Electronics/MCU.kicad_sch (KiCad schematic)
At the start: 11 parts, among them J301 UART, J302 I2C, U301 74HC86, U302 74AHC08

Commit message: Manufacturing commit of PCB
Connections:
- net HIN A: now also A301.12 (D9); no longer A301.6 (D3)
- net HIN B: now also A301.14 (MOSI); no longer A301.13 (D10)
- net LIN A: now also A301.13 (D10); no longer A301.14 (MOSI)
- net LIN B: now also A301.6 (D3); no longer A301.12 (D9)
- net CTRL C: now reaches A301.16 (SCK)
- net LIMIT C renamed CTRL A
- no-connect marks 8 -> 7
