File: Electronics/Power.kicad_sch (KiCad schematic)
At the start: 26 parts, among them U400 R-78C3.3-1.0, U401 R-78C5.0-1.0, U402 R-78C15-1.0

Commit message: Added STM32 Code for BLDC controller
Parts:
- added FID401, FID402, FID403: Fiducial, Fiducial:Fiducial_1.5mm_Mask3mm, symbol Mechanical:Fiducial
Changed lines of the file:
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@@
+    )
+  )
+  (symbol (lib_id "Mechanical:Fiducial") (at 90.805 190.5 0) (unit 1)
+    (in_bom yes) (on_board yes) (fields_autoplaced)
+    (property "Reference" "FID403" (id 0) (at 92.964 189.5915 0)
+      (effects (font (size 1.27 1.27)) (justify left))
+    )
+    (property "Value" "Fiducial" (id 1) (at 92.964 192.3666 0)
+      (effects (font (size 1.27 1.27)) (justify left))
+    )
+    (property "Footprint" "Fiducial:Fiducial_1.5mm_Mask3mm" (id 2) (at 90.805 190.5 0)
+      (effects (font (size 1.27 1.27)) hide)
+    )
+    (property "Datasheet" "~" (id 3) (at 90.805 190.5 0)
+      (effects (font (size 1.27 1.27)) hide)
     )
   )
@@
     (pin "2")
   )
+  (symbol (lib_id "Mechanical:Fiducial") (at 90.805 179.07 0) (unit 1)
+    (in_bom yes) (on_board yes) (fields_autoplaced)
+    (property "Reference" "FID401" (id 0) (at 92.964 178.1615 0)
+      (effects (font (size 1.27 1.27)) (justify left))
+    )
+    (property "Value" "Fiducial" (id 1) (at 92.964 180.9366 0)
+      (effects (font (size 1.27 1.27)) (justify left))
+    )
+    (property "Footprint" "Fiducial:Fiducial_1.5mm_Mask3mm" (id 2) (at 90.805 179.07 0)
+      (effects (font (size 1.27 1.27)) hide)
+    )
+    (property "Datasheet" "~" (id 3) (at 90.805 179.07 0)
+      (effects (font (size 1.27 1.27)) hide)
+    )
+  )
   (symbol (lib_id "Device:C") (at 209.55 59.69 0) (unit 1)
     (in_bom yes) (on_board yes) (fields_autoplaced)
@@
     (pin "1")
   )
+  (symbol (lib_id "Mechanical:Fiducial") (at 90.805 184.785 0) (unit 1)
+    (in_bom yes) (on_board yes) (fields_autoplaced)
+    (property "Reference" "FID402" (id 0) (at 92.964 183.8765 0)
+      (effects (font (size 1.27 1.27)) (justify left))
+    )
+    (property "Value" "Fiducial" (id 1) (at 92.964 186.6516 0)
+      (effects (font (size 1.27 1.27)) (justify left))
+    )
+    (property "Footprint" "Fiducial:Fiducial_1.5mm_Mask3mm" (id 2) (at 90.805 184.785 0)
+      (effects (font (size 1.27 1.27)) hide)
+    )
+    (property "Datasheet" "~" (id 3) (at 90.805 184.785 0)
+      (effects (font (size 1.27 1.27)) hide)
+    )
+  )
   (symbol (lib_name "MountingHole_1") (lib_id "Mechanical:MountingHole") (at 114.3 182.88 0) (unit 1)
