File: Electronics/controller.kicad_sch (KiCad schematic)
At the start: 0 parts

Commit message: Layout improvements
Signed-off-by: Aki Kuusela <git@findersee.fi>
Other:
- sheet Connectors ports: added Over Current; removed none
- sheet MCU ports: added LIMIT MCU 1, LIMIT MCU 2, OCP; removed LIMIT 1, LIMIT 2
- company: (none) -> findersee.fi
- title: (none) -> Motor Controller
Changed lines of the file:
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@@
 (kicad_sch (version 20211123) (generator eeschema)
   (paper "A4")
+  (title_block
+    (title "Motor Controller")
+    (date "2022-02-18")
+    (rev "1.0")
+    (company "findersee.fi")
+  )
   (junction (at 156.21 76.2) (diameter 0) (color 0 0 0 0)
   )
@@
   )
   (wire (pts (xy 83.82 134.62) (xy 163.83 134.62))
+    (stroke (width 0) (type default) (color 0 0 0 0))
+  )
+  (wire (pts (xy 83.82 146.05) (xy 163.83 146.05))
     (stroke (width 0) (type default) (color 0 0 0 0))
   )
@@
     )
   )
-  (sheet (at 163.83 71.12) (size 34.29 75.565) (fields_autoplaced)
+  (sheet (at 163.83 71.12) (size 34.29 78.105) (fields_autoplaced)
     (stroke (width 0.1524) (type solid) (color 0 0 0 0))
     (fill (color 0 0 0 0.0000))
@@
       (effects (font (size 1.27 1.27)) (justify left bottom))
     )
-    (property "Sheet file" "Connectors.kicad_sch" (id 1) (at 163.83 147.2696 0)
+    (property "Sheet file" "Connectors.kicad_sch" (id 1) (at 163.83 149.8096 0)
       (effects (font (size 1.27 1.27)) (justify left top))
     )
@@
       (effects (font (size 1.27 1.27)) (justify left))
     )
-  )
-  (sheet (at 50.8 71.12) (size 33.02 76.2) (fields_autoplaced)
+    (pin "Over Current" output (at 163.83 146.05 180)
+      (effects (font (size 1.27 1.27)) (justify left))
+    )
+  )
+  (sheet (at 50.8 71.12) (size 33.02 79.375) (fields_autoplaced)
     (stroke (width 0.1524) (type solid) (color 0 0 0 0))
     (fill (color 0 0 0 0.0000))
@@
       (effects (font (size 1.27 1.27)) (justify left bottom))
     )
-    (property "Sheet file" "MCU.kicad_sch" (id 1) (at 50.8 147.9046 0)
+    (property "Sheet file" "MCU.kicad_sch" (id 1) (at 50.8 151.0796 0)
       (effects (font (size 1.27 1.27)) (justify left top))
     )
@@
       (effects (font (size 1.27 1.27)) (justify right))
     )
-    (pin "LIMIT 1" bidirectional (at 83.82 76.2 0)
+    (pin "LIMIT MCU 1" bidirectional (at 83.82 76.2 0)
       (effects (font (size 1.27 1.27)) (justify right))
     )
@@
       (effects (font (size 1.27 1.27)) (justify right))
     )
-    (pin "LIMIT 2" bidirectional (at 83.82 78.74 0)
+    (pin "LIMIT MCU 2" bidirectional (at 83.82 78.74 0)
       (effects (font (size 1.27 1.27)) (justify right))
     )
@@
     )
     (pin "Latch Reset" output (at 83.82 143.51 0)
+      (effects (font (size 1.27 1.27)) (justify right))
+    )
+    (pin "OCP" input (at 83.82 146.05 0)
       (effects (font (size 1.27 1.27)) (justify right))
     )
@@
   )
   (symbol_instances
+    (path "/aa31faa7-1bf1-4443-8396-f678eeba3772/bad63119-e054-4a62-a294-b2922b556d5c"
+      (reference "#FLG0101") (unit 1) (value "PWR_FLAG") (footprint "")
+    )
     (path "/aa31faa7-1bf1-4443-8396-f678eeba3772/628b297f-f130-4ba6-8d18-c2f1845b4947"
       (reference "#FLG0103") (unit 1) (value "PWR_FLAG") (footprint "")
@@
       (reference "#PWR0113") (unit 1) (value "VCC") (footprint "")
     )
+    (path "/f1c4a73a-91cc-421a-b2f5-51b0bd7a9f21/3d442bb6-0b90-46de-bf54-bae2e37773e3"
+      (reference "#PWR0114") (unit 1) (value "+3V3") (footprint "")
+    )
     (path "/aa31faa7-1bf1-4443-8396-f678eeba3772/ed52b762-9670-48f1-b85a-1d5b2cfb4325"
       (reference "#PWR0115") (unit 1) (value "+3V3") (footprint "")
@@
       (reference "#PWR0144") (unit 1) (value "GND") (footprint "")
     )
+    (path "/f1c4a73a-91cc-421a-b2f5-51b0bd7a9f21/c9e38c04-94ca-441b-876a-1034a67ff213"
+      (reference "#PWR0145") (unit 1) (value "GND") (footprint "")
+    )
+    (path "/f1c4a73a-91cc-421a-b2f5-51b0bd7a9f21/bb7efc93-5239-40f8-b1ab-d7d884fc95bb"
+      (reference "#PWR0146") (unit 1) (value "+3V3") (footprint "")
+    )
+    (path "/aa31faa7-1bf1-4443-8396-f678eeba3772/35aaf033-7e2f-4a4d-8f41-984e9a637950"
+      (reference "#PWR0147") (unit 1) (value "+3V3") (footprint "")
+    )
+    (path "/f1c4a73a-91cc-421a-b2f5-51b0bd7a9f21/9922df6a-2872-47cb-99a9-5b361d86eb09"
+      (reference "#PWR0148") (unit 1) (value "GND") (footprint "")
+    )
     (path "/f1c4a73a-91cc-421a-b2f5-51b0bd7a9f21/50c34630-6674-4756-a8e8-c57a351dbf5d"
       (reference "#PWR0301") (unit 1) (value "GND") (footprint "")
@@
       (reference "#PWR0518") (unit 1) (value "VDD") (footprint "")
     )
-    (path "/aa31faa7-1bf1-4443-8396-f678eeba3772/041b37ec-4c82-454f-b375-b6208bb03fb7"
-      (reference "#PWR0519") (unit 1) (value "GND") (footprint "")
-    )
     (path "/aa31faa7-1bf1-4443-8396-f678eeba3772/ff23efb8-153d-4afb-b85c-c4e507f3b942"
       (reference "#PWR0520") (unit 1) (value "GND") (footprint "")
@@
       (reference "#PWR0523") (unit 1) (value "VDD") (footprint "")
     )
-    (path "/f1c4a73a-91cc-421a-b2f5-51b0bd7a9f21/3d442bb6-0b90-46de-bf54-bae2e37773e3"
-      (reference "#PWR?") (unit 1) (value "+3V3") (footprint "")
-    )
     (path "/f1c4a73a-91cc-421a-b2f5-51b0bd7a9f21/5521e049-8492-4615-a629-fed11f1f3e70"
       (reference "A301") (unit 1) (value "Arduino_Nano_Every") (footprint "Module:Arduino_Nano")
@@
       (reference "J301") (unit 1) (value "UART") (footprint "Connector_PinHeader_2.54mm:PinHeader_1x03_P2.54mm_Vertical")
     )
+    (path "/f1c4a73a-91cc-421a-b2f5-51b0bd7a9f21/beca0a7f-e627-41bb-b94d-b67d3a8b20e0"
+      (reference "J302") (unit 1) (value "I2C") (footprint "Connector_PinHeader_2.54mm:PinHeader_1x04_P2.54mm_Vertical")
+    )
     (path "/aa31faa7-1bf1-4443-8396-f678eeba3772/45e2ff1d-a830-4e8c-8bc6-8947bd353757"
       (reference "J501") (unit 1) (value "Switches") (footprint "TerminalBlock:TerminalBlock_bornier-6_P5.08mm")
@@
     )
     (path "/4be341a8-7d6b-4e6c-8950-2eaf98627d00/f91bcd7d-e175-40b2-96c1-31a50d044668"
-      (reference "U201") (unit 1) (value "74AHC08") (footprint "Package_SO:SSOP-14_5.3x6.2mm_P0.65mm")
+      (reference "U201") (unit 1) (value "74LS08") (footprint "Package_SO:SO-14_3.9x8.65mm_P1.27mm")
     )
     (path "/4be341a8-7d6b-4e6c-8950-2eaf98627d00/3437108d-25a1-40a2-8fab-34d22c11db3c"
-      (reference "U201") (unit 2) (value "74AHC08") (footprint "Package_SO:SSOP-14_5.3x6.2mm_P0.65mm")
+      (reference "U201") (unit 2) (value "74LS08") (footprint "Package_SO:SO-14_3.9x8.65mm_P1.27mm")
     )
     (path "/4be341a8-7d6b-4e6c-8950-2eaf98627d00/9327f1aa-dbea-4fcc-bdc3-4fd2e32fe928"
-      (reference "U201") (unit 3) (value "74AHC08") (footprint "Package_SO:SSOP-14_5.3x6.2mm_P0.65mm")
+      (reference "U201") (unit 3) (value "74LS08") (footprint "Package_SO:SO-14_3.9x8.65mm_P1.27mm")
     )
     (path "/4be341a8-7d6b-4e6c-8950-2eaf98627d00/b533a8b5-764b-46ef-842e-43cd02dc1193"
-      (reference "U201") (unit 4) (value "74AHC08") (footprint "Package_SO:SSOP-14_5.3x6.2mm_P0.65mm")
+      (reference "U201") (unit 4) (value "74LS08") (footprint "Package_SO:SO-14_3.9x8.65mm_P1.27mm")
     )
     (path "/4be341a8-7d6b-4e6c-8950-2eaf98627d00/a700115e-151f-44f9-809a-cb5c5c50120b"
-      (reference "U201") (unit 5) (value "74AHC08") (footprint "Package_SO:SSOP-14_5.3x6.2mm_P0.65mm")
+      (reference "U201") (unit 5) (value "74LS08") (footprint "Package_SO:SO-14_3.9x8.65mm_P1.27mm")
     )
     (path "/4be341a8-7d6b-4e6c-8950-2eaf98627d00/6c64cdd5-b388-4d44-a385-adcffa867cd6"

Commit message: Manufacturing commit of PCB
Other:
- sheet Hbridge ports: added A CTRL, C CTRL; removed C LIMIT
- sheet MCU ports: added CTRL A, CTRL C; removed LIMIT C
Changed lines of the file:
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@@
   (title_block
     (title "Motor Controller")
-    (date "2022-02-18")
+    (date "2022-02-20")
     (rev "1.0")
     (company "findersee.fi")
@@
     (stroke (width 0) (type default) (color 0 0 0 0))
   )
+  (wire (pts (xy 83.82 121.285) (xy 115.57 121.285))
+    (stroke (width 0) (type default) (color 0 0 0 0))
+  )
   (wire (pts (xy 83.82 90.17) (xy 115.57 90.17))
     (stroke (width 0) (type default) (color 0 0 0 0))
@@
     (stroke (width 0) (type default) (color 0 0 0 0))
   )
-  (wire (pts (xy 83.82 121.92) (xy 115.57 121.92))
-    (stroke (width 0) (type default) (color 0 0 0 0))
-  )
   (wire (pts (xy 83.82 92.71) (xy 115.57 92.71))
+    (stroke (width 0) (type default) (color 0 0 0 0))
+  )
+  (wire (pts (xy 83.82 123.825) (xy 115.57 123.825))
     (stroke (width 0) (type default) (color 0 0 0 0))
   )
@@
       (effects (font (size 1.27 1.27)) (justify left))
     )
-    (pin "C LIMIT" input (at 115.57 121.92 180)
-      (effects (font (size 1.27 1.27)) (justify left))
-    )
     (pin "C_OUT" output (at 148.59 115.57 0)
       (effects (font (size 1.27 1.27)) (justify right))
+    )
+    (pin "A CTRL" input (at 115.57 121.285 180)
+      (effects (font (size 1.27 1.27)) (justify left))
+    )
+    (pin "C CTRL" input (at 115.57 123.825 180)
+      (effects (font (size 1.27 1.27)) (justify left))
     )
   )
@@
       (effects (font (size 1.27 1.27)) (justify right))
     )
-    (pin "LIMIT C" output (at 83.82 121.92 0)
-      (effects (font (size 1.27 1.27)) (justify right))
-    )
     (pin "HALL C" input (at 83.82 132.08 0)
       (effects (font (size 1.27 1.27)) (justify right))
@@
     )
     (pin "OCP" input (at 83.82 146.05 0)
+      (effects (font (size 1.27 1.27)) (justify right))
+    )
+    (pin "CTRL A" output (at 83.82 121.285 0)
+      (effects (font (size 1.27 1.27)) (justify right))
+    )
+    (pin "CTRL C" output (at 83.82 123.825 0)
       (effects (font (size 1.27 1.27)) (justify right))
     )
@@
       (reference "#FLG0101") (unit 1) (value "PWR_FLAG") (footprint "")
     )
+    (path "/54222278-f439-4dd5-b7a2-082afad1f322/f6921110-041c-46c2-b6eb-a407fb1aa69a"
+      (reference "#FLG0102") (unit 1) (value "PWR_FLAG") (footprint "")
+    )
     (path "/aa31faa7-1bf1-4443-8396-f678eeba3772/628b297f-f130-4ba6-8d18-c2f1845b4947"
       (reference "#FLG0103") (unit 1) (value "PWR_FLAG") (footprint "")
@@
       (reference "#PWR0108") (unit 1) (value "GND") (footprint "")
     )
-    (path "/4be341a8-7d6b-4e6c-8950-2eaf98627d00/e5832edd-5830-4dae-ac25-40e4a20a44a4"
-      (reference "#PWR0109") (unit 1) (value "+3V3") (footprint "")
+    (path "/54222278-f439-4dd5-b7a2-082afad1f322/ecfd91bf-b1e1-4cae-b358-b219815c0f8c"
+      (reference "#PWR0109") (unit 1) (value "GND") (footprint "")
     )
     (path "/4be341a8-7d6b-4e6c-8950-2eaf98627d00/08eab6fd-7e22-49a0-8e3f-2332d9b3f101"
@@
       (reference "#PWR0148") (unit 1) (value "GND") (footprint "")
     )
+    (path "/4be341a8-7d6b-4e6c-8950-2eaf98627d00/0542db7c-c6c7-4c1c-927b-967200d43085"
+      (reference "#PWR0201") (unit 1) (value "+3V3") (footprint "")
+    )
+    (path "/4be341a8-7d6b-4e6c-8950-2eaf98627d00/fd41cf1d-a9c6-472a-ac5e-563f344b1836"
+      (reference "#PWR0202") (unit 1) (value "GND") (footprint "")
+    )
+    (path "/4be341a8-7d6b-4e6c-8950-2eaf98627d00/ec5d6c18-2d13-4817-9b73-5743b856d2f7"
+      (reference "#PWR0203") (unit 1) (value "GND") (footprint "")
+    )
+    (path "/4be341a8-7d6b-4e6c-8950-2eaf98627d00/f5b24097-daac-425b-aeb5-981d18a2af43"
+      (reference "#PWR0205") (unit 1) (value "GND") (footprint "")
+    )
     (path "/f1c4a73a-91cc-421a-b2f5-51b0bd7a9f21/50c34630-6674-4756-a8e8-c57a351dbf5d"
       (reference "#PWR0301") (unit 1) (value "GND") (footprint "")
@@
       (reference "#PWR0307") (unit 1) (value "GND") (footprint "")
     )
+    (path "/54222278-f439-4dd5-b7a2-082afad1f322/e164c5cf-6f34-473c-b0cf-38584657ff38"
+      (reference "#PWR0401") (unit 1) (value "GND") (footprint "")
+    )
+    (path "/54222278-f439-4dd5-b7a2-082afad1f322/8b7ebfb2-4d2a-4805-ad8a-550eabb9d39a"
+      (reference "#PWR0402") (unit 1) (value "+3V3") (footprint "")
+    )
     (path "/aa31faa7-1bf1-4443-8396-f678eeba3772/54a6ba8f-29f1-4bab-8719-7f7d7772629b"
       (reference "#PWR0501") (unit 1) (value "VDD") (footprint "")
@@
     )
     (path "/4be341a8-7d6b-4e6c-8950-2eaf98627d00/9ac87bec-e4b1-4c3d-91ab-a0d0ce1314ca"
-      (reference "C201") (unit 1) (value "C") (footprint "Capacitor_SMD:C_0603_1608Metric_Pad1.08x0.95mm_HandSolder")
+      (reference "C201") (unit 1) (value "100n") (footprint "Capacitor_SMD:C_0603_1608Metric_Pad1.08x0.95mm_HandSolder")
     )
     (path "/4be341a8-7d6b-4e6c-8950-2eaf98627d00/05641547-6b29-412b-93aa-3dab1a224e19"
@@
       (reference "C210") (unit 1) (value "100u") (footprint "Findersee_parts:CP_Radial_D12.5mm_P3.5-5.0mm")
     )
+    (path "/4be341a8-7d6b-4e6c-8950-2eaf98627d00/e6ff8a54-3da3-44c0-801d-dc3a3c41b1d6"
+      (reference "C211") (unit 1) (value "100n") (footprint "Capacitor_SMD:C_0603_1608Metric_Pad1.08x0.95mm_HandSolder")
+    )
     (path "/f1c4a73a-91cc-421a-b2f5-51b0bd7a9f21/40deb473-9f31-47ca-b074-23c81d2e8441"
       (reference "C301") (unit 1) (value "100n") (footprint "Capacitor_SMD:C_0603_1608Metric_Pad1.08x0.95mm_HandSolder")
@@
       (reference "C408") (unit 1) (value "10u") (footprint "Resistor_SMD:R_0805_2012Metric_Pad1.20x1.40mm_HandSolder")
     )
+    (path "/54222278-f439-4dd5-b7a2-082afad1f322/308d195c-aee2-41e4-9c94-887d2b588f5f"
+      (reference "C409") (unit 1) (value "4u7") (footprint "Resistor_SMD:R_0805_2012Metric_Pad1.20x1.40mm_HandSolder")
+    )
+    (path "/54222278-f439-4dd5-b7a2-082afad1f322/50bec952-6677-4866-8c61-a3afd6832d0a"
+      (reference "C410") (unit 1) (value "100n") (footprint "Capacitor_SMD:C_0603_1608Metric_Pad1.08x0.95mm_HandSolder")
+    )
+    (path "/54222278-f439-4dd5-b7a2-082afad1f322/b8226827-88d0-4c05-ad8b-30a50cfef5fc"
+      (reference "C411") (unit 1) (value "100n") (footprint "Capacitor_SMD:C_0603_1608Metric_Pad1.08x0.95mm_HandSolder")
+    )
+    (path "/54222278-f439-4dd5-b7a2-082afad1f322/f6df09ab-b40f-4766-90b2-9080ea5f067f"
+      (reference "C412") (unit 1) (value "10u") (footprint "Resistor_SMD:R_0805_2012Metric_Pad1.20x1.40mm_HandSolder")
+    )
     (path "/aa31faa7-1bf1-4443-8396-f678eeba3772/71936a86-c448-4f2c-8383-8911972fcd6f"
       (reference "C501") (unit 1) (value "100n") (footprint "Capacitor_SMD:C_0603_1608Metric_Pad1.08x0.95mm_HandSolder")
@@
       (reference "R214") (unit 1) (value "0") (footprint "Resistor_SMD:R_0603_1608Metric_Pad0.98x0.95mm_HandSolder")
     )
+    (path "/4be341a8-7d6b-4e6c-8950-2eaf98627d00/baf807da-7e74-4d42-9348-a65f03d3be71"
+      (reference "R215") (unit 1) (value "0") (footprint "Resistor_SMD:R_0603_1608Metric_Pad0.98x0.95mm_HandSolder")
+    )
+    (path "/4be341a8-7d6b-4e6c-8950-2eaf98627d00/7ac77941-e158-4e6c-93b5-cae86a5cfa0b"
+      (reference "R216") (unit 1) (value "0") (footprint "Resistor_SMD:R_0603_1608Metric_Pad0.98x0.95mm_HandSolder")
+    )
+    (path "/4be341a8-7d6b-4e6c-8950-2eaf98627d00/920cdc78-02fd-4c87-96e7-8fc61fe49be8"
+      (reference "R217") (unit 1) (value "0") (footprint "Resistor_SMD:R_0603_1608Metric_Pad0.98x0.95mm_HandSolder")
+    )
+    (path "/4be341a8-7d6b-4e6c-8950-2eaf98627d00/b12ec3d0-b14a-4b95-8a46-86d850d7159e"
+      (reference "R218") (unit 1) (value "0") (footprint "Resistor_SMD:R_0603_1608Metric_Pad0.98x0.95mm_HandSolder")
+    )
     (path "/f1c4a73a-91cc-421a-b2f5-51b0bd7a9f21/e6ab23dd-7e4f-4d27-ac66-ac20059da534"
       (reference "R301") (unit 1) (value "0") (footprint "Resistor_SMD:R_0603_1608Metric_Pad0.98x0.95mm_HandSolder")
@@
       (reference "U204") (unit 1) (value "IR2101") (footprint "Package_SO:SO-8_3.9x4.9mm_P1.27mm")
     )
+    (path "/4be341a8-7d6b-4e6c-8950-2eaf98627d00/2f8c467f-c568-40e7-b45f-c00d2d7d7568"
+      (reference "U205") (unit 1) (value "74LS08") (footprint "Package_SO:SO-14_3.9x8.65mm_P1.27mm")
+    )
+    (path "/4be341a8-7d6b-4e6c-8950-2eaf98627d00/2b6f74da-a2a1-43af-87b2-4c93c7196085"
+      (reference "U205") (unit 2) (value "74LS08") (footprint "Package_SO:SO-14_3.9x8.65mm_P1.27mm")
+    )
+    (path "/4be341a8-7d6b-4e6c-8950-2eaf98627d00/f7a10e84-4b9e-4236-82e0-f447fb7c9e64"
+      (reference "U205") (unit 3) (value "74LS08") (footprint "Package_SO:SO-14_3.9x8.65mm_P1.27mm")
+    )
+    (path "/4be341a8-7d6b-4e6c-8950-2eaf98627d00/f270cd20-37ed-4b16-a457-26dd61adffd2"
+      (reference "U205") (unit 4) (value "74LS08") (footprint "Package_SO:SO-14_3.9x8.65mm_P1.27mm")
+    )
+    (path "/4be341a8-7d6b-4e6c-8950-2eaf98627d00/a24024d6-1087-4aaf-a488-d7c5ab6d424b"
+      (reference "U205") (unit 5) (value "74LS08") (footprint "Package_SO:SO-14_3.9x8.65mm_P1.27mm")
+    )
     (path "/f1c4a73a-91cc-421a-b2f5-51b0bd7a9f21/5aa7be24-0bc1-4162-bdcc-fbe34438489e"
       (reference "U301") (unit 1) (value "74HC86") (footprint "Package_SO:SO-14_3.9x8.65mm_P1.27mm")
@@
       (reference "U302") (unit 5) (value "74AHC08") (footprint "Package_SO:SSOP-14_5.3x6.2mm_P0.65mm")
     )
+    (path "/54222278-f439-4dd5-b7a2-082afad1f322/7317d372-cc09-43b6-af1d-e0fbdfd9b47c"
+      (reference "U400") (unit 1) (value "R-78C3.3-1.0") (footprint "Converter_DCDC:Converter_DCDC_RECOM_R-78E-0.5_THT")
+    )
     (path "/54222278-f439-4dd5-b7a2-082afad1f322/0293f46b-77a7-4330-bbe8-30f00dcdc421"
